Commit message: URDF: all six joints

File: urdf/so101.urdf (robot description, URDF)
Before this commit: robot so101, 4 links, 3 joints
Links:
- added link gripper_link; visual box size=0.03 0.03 0.03
- added link moving_jaw_so101_v1_link; visual box size=0.03 0.03 0.03
- added link wrist_link; visual box size=0.03 0.03 0.03
Joints:
- added joint gripper: type revolute, parent gripper_link, child moving_jaw_so101_v1_link, origin xyz=0.0202 0.0188 -0.0234 rpy=1.5708 -5.24284e-08 -1.41553e-15, axis 0 0 1, limit lower=-0.174533 upper=1.74533 effort=10 velocity=5
- added joint wrist_flex: type revolute, parent lower_arm_link, child wrist_link, origin xyz=-0.1349 0.0052 3.62355e-17 rpy=0.0 0.0 -1.5708, axis 0 0 1, limit lower=-1.65806 upper=1.65806 effort=10 velocity=5
- added joint wrist_roll: type revolute, parent wrist_link, child gripper_link, origin xyz=5.55112e-17 -0.0611 0.0181 rpy=1.5708 0.0486795 3.14159, axis 0 0 1, limit lower=-2.74385 upper=2.84121 effort=10 velocity=5
